File: hardware/rgbeep.sch (KiCad schematic (older format))
At the start: 22 parts, among them SW1 SW_PUSH, SW2 SW_PUSH, SW3 SW_PUSH, SW4 SW_PUSH, U1 APA102, U10 APA102, U11 APA102, U12 APA102, U13 APA102, U14 APA102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

Commit message: Select footprints for parts.
Parts:
- SW1, SW2, SW3, SW4: footprint (none) -> CrumpPrints:6x6mm_pushbutton
- U1, U10, U11, U12, U13, U14, U15, U16, U2, U3, U4, U5, U6, U7, U8, U9: footprint (none) -> CrumpPrints:APA102
- U17: footprint (none) -> CrumpPrints:D1_mini
- U18: footprint (none) -> Housings_SOIC:SOIC-14_3.9x8.7mm_Pitch1.27mm
Changed lines of the file:
@@
 F 0 "U1" H 1650 1300 60  0000 C CNN
 F 1 "APA102" H 1750 700 60  0000 C CNN
-F 2 "" H 1850 550 60  0000 C CNN
+F 2 "CrumpPrints:APA102" H 1850 550 60  0001 C CNN
 F 3 "" H 1850 550 60  0000 C CNN
 	1    1850 1000
@@
 F 0 "U2" H 2700 1300 60  0000 C CNN
 F 1 "APA102" H 2800 700 60  0000 C CNN
-F 2 "" H 2900 550 60  0000 C CNN
+F 2 "CrumpPrints:APA102" H 2900 550 60  0001 C CNN
 F 3 "" H 2900 550 60  0000 C CNN
 	1    2900 1000
@@
 F 0 "U3" H 3750 1300 60  0000 C CNN
 F 1 "APA102" H 3850 700 60  0000 C CNN
-F 2 "" H 3950 550 60  0000 C CNN
+F 2 "CrumpPrints:APA102" H 3950 550 60  0001 C CNN
 F 3 "" H 3950 550 60  0000 C CNN
 	1    3950 1000
@@
 F 0 "U4" H 4800 1300 60  0000 C CNN
 F 1 "APA102" H 4900 700 60  0000 C CNN
-F 2 "" H 5000 550 60  0000 C CNN
+F 2 "CrumpPrints:APA102" H 5000 550 60  0001 C CNN
 F 3 "" H 5000 550 60  0000 C CNN
 	1    5000 1000
@@
 F 0 "U5" H 5850 1300 60  0000 C CNN
 F 1 "APA102" H 5950 700 60  0000 C CNN
-F 2 "" H 6050 550 60  0000 C CNN
+F 2 "CrumpPrints:APA102" H 6050 550 60  0001 C CNN
 F 3 "" H 6050 550 60  0000 C CNN
 	1    6050 1000
@@
 F 0 "U6" H 6900 1300 60  0000 C CNN
 F 1 "APA102" H 7000 700 60  0000 C CNN
-F 2 "" H 7100 550 60  0000 C CNN
+F 2 "CrumpPrints:APA102" H 7100 550 60  0001 C CNN
 F 3 "" H 7100 550 60  0000 C CNN
 	1    7100 1000
@@
 F 0 "U7" H 7950 1300 60  0000 C CNN
 F 1 "APA102" H 8050 700 60  0000 C CNN
-F 2 "" H 8150 550 60  0000 C CNN
+F 2 "CrumpPrints:APA102" H 8150 550 60  0001 C CNN
 F 3 "" H 8150 550 60  0000 C CNN
 	1    8150 1000
@@
 F 0 "U8" H 9000 1300 60  0000 C CNN
 F 1 "APA102" H 9100 700 60  0000 C CNN
-F 2 "" H 9200 550 60  0000 C CNN
+F 2 "CrumpPrints:APA102" H 9200 550 60  0001 C CNN
 F 3 "" H 9200 550 60  0000 C CNN
 	1    9200 1000
@@
 F 0 "U9" H 1650 2350 60  0000 C CNN
 F 1 "APA102" H 1750 1750 60  0000 C CNN
-F 2 "" H 1850 1600 60  0000 C CNN
+F 2 "CrumpPrints:APA102" H 1850 1600 60  0001 C CNN
 F 3 "" H 1850 1600 60  0000 C CNN
 	1    1850 2050
@@
 F 0 "U10" H 2700 2350 60  0000 C CNN
 F 1 "APA102" H 2800 1750 60  0000 C CNN
-F 2 "" H 2900 1600 60  0000 C CNN
+F 2 "CrumpPrints:APA102" H 2900 1600 60  0001 C CNN
 F 3 "" H 2900 1600 60  0000 C CNN
 	1    2900 2050
@@
 F 0 "U11" H 3750 2350 60  0000 C CNN
 F 1 "APA102" H 3850 1750 60  0000 C CNN
-F 2 "" H 3950 1600 60  0000 C CNN
+F 2 "CrumpPrints:APA102" H 3950 1600 60  0001 C CNN
 F 3 "" H 3950 1600 60  0000 C CNN
 	1    3950 2050
@@
 F 0 "U12" H 4800 2350 60  0000 C CNN
 F 1 "APA102" H 4900 1750 60  0000 C CNN
-F 2 "" H 5000 1600 60  0000 C CNN
+F 2 "CrumpPrints:APA102" H 5000 1600 60  0001 C CNN
 F 3 "" H 5000 1600 60  0000 C CNN
 	1    5000 2050
@@
 F 0 "U13" H 5850 2350 60  0000 C CNN
 F 1 "APA102" H 5950 1750 60  0000 C CNN
-F 2 "" H 6050 1600 60  0000 C CNN
+F 2 "CrumpPrints:APA102" H 6050 1600 60  0001 C CNN
 F 3 "" H 6050 1600 60  0000 C CNN
 	1    6050 2050
@@
 F 0 "U14" H 6900 2350 60  0000 C CNN
 F 1 "APA102" H 7000 1750 60  0000 C CNN
-F 2 "" H 7100 1600 60  0000 C CNN
+F 2 "CrumpPrints:APA102" H 7100 1600 60  0001 C CNN
 F 3 "" H 7100 1600 60  0000 C CNN
 	1    7100 2050
@@
 F 0 "U15" H 7950 2350 60  0000 C CNN
 F 1 "APA102" H 8050 1750 60  0000 C CNN
-F 2 "" H 8150 1600 60  0000 C CNN
+F 2 "CrumpPrints:APA102" H 8150 1600 60  0001 C CNN
 F 3 "" H 8150 1600 60  0000 C CNN
 	1    8150 2050
@@
 F 0 "U16" H 9000 2350 60  0000 C CNN
 F 1 "APA102" H 9100 1750 60  0000 C CNN
-F 2 "" H 9200 1600 60  0000 C CNN
+F 2 "CrumpPrints:APA102" H 9200 1600 60  0001 C CNN
 F 3 "" H 9200 1600 60  0000 C CNN
 	1    9200 2050
@@
 F 0 "U17" H 1900 2600 60  0000 C CNN
 F 1 "Wemos_D1_Mini" H 1900 3700 60  0000 C CNN
-F 2 "" H 1900 3300 60  0001 C CNN
+F 2 "CrumpPrints:D1_mini" H 1900 3300 60  0001 C CNN
 F 3 "" H 1900 3300 60  0001 C CNN
 	1    1900 3300
@@
 F 0 "U18" H 4150 2750 60  0000 C CNN
 F 1 "SN74AHCT125" H 4150 4200 60  0000 C CNN
-F 2 "" H 4150 3550 60  0001 C CNN
+F 2 "Housings_SOIC:SOIC-14_3.9x8.7mm_Pitch1.27mm" H 4150 3550 60  0001 C CNN
 F 3 "" H 4150 3550 60  0001 C CNN
 	1    4150 3550
@@
 F 0 "SW1" H 5950 3160 50  0000 C CNN
 F 1 "SW_PUSH" H 5800 2970 50  0000 C CNN
-F 2 "" H 5800 3050 50  0000 C CNN
+F 2 "CrumpPrints:6x6mm_pushbutton" H 5800 3050 50  0001 C CNN
 F 3 "" H 5800 3050 50  0000 C CNN
 	1    5800 3050
@@
 F 0 "SW2" H 5950 3460 50  0000 C CNN
 F 1 "SW_PUSH" H 5800 3270 50  0000 C CNN
-F 2 "" H 5800 3350 50  0000 C CNN
+F 2 "CrumpPrints:6x6mm_pushbutton" H 5800 3350 50  0001 C CNN
 F 3 "" H 5800 3350 50  0000 C CNN
 	1    5800 3350
@@
 F 0 "SW3" H 5950 3760 50  0000 C CNN
 F 1 "SW_PUSH" H 5800 3570 50  0000 C CNN
-F 2 "" H 5800 3650 50  0000 C CNN
+F 2 "CrumpPrints:6x6mm_pushbutton" H 5800 3650 50  0001 C CNN
 F 3 "" H 5800 3650 50  0000 C CNN
 	1    5800 3650
@@
 F 0 "SW4" H 5950 4060 50  0000 C CNN
 F 1 "SW_PUSH" H 5800 3870 50  0000 C CNN
-F 2 "" H 5800 3950 50  0000 C CNN
+F 2 "CrumpPrints:6x6mm_pushbutton" H 5800 3950 50  0001 C CNN
 F 3 "" H 5800 3950 50  0000 C CNN
 	1    5800 3950
